File: EsquemaEletrico/ProjetoFinalSEMB.kicad_sch (KiCad schematic)
At the start: 52 parts, among them SW1 SW_Push, SW2 SW_Push

Commit message: Projeto final completo
Parts:
- IC_OA1: footprint Footprints:SOP50P326X110-14N -> Footprints:SOP65P640X120-14N
- R1, R10, R11, R12, R13, R14, R15, R16, R2, R3, R6, R7, R8: footprint Footprints:H2C_H2R -> Footprints:ERJ1T__2512_
- R17, R18, R19, R20, R21, R22: footprint Footprints:H2C_H2R -> Footprints:ERJL12__1812_
- R23, R24: value 4.7K -> 2.2K; footprint Footprints:H2C_H2R -> Footprints:ERJ1T__2512_
Connections:
- net I2C_SCL: now also MIcrocontroler1.45 (PB8); no longer MIcrocontroler1.42 (PB6)
- net PWM: now also MIcrocontroler1.19 (PB1); no longer MIcrocontroler1.40 (PB4)
- net SD_DAT2: now also R17.1; no longer R17.2
- net SD_DET_B: now also MIcrocontroler1.25 (PB12); no longer MIcrocontroler1.10 (PA0)
- net at MicroSD1.1 (DAT2): now also R17.2; no longer R17.1
Other:
- note added: "Power Flags"
- moved on the sheet: MIcrocontroler1, R17, R4, R5
